File: jack-boards/jack-boards.kicad_pcb (KiCad board)
At the start: 2 copper layers, 9 parts, among them J1 AudioJack3_Ground_Switch, J2 AudioJack3_Ground_Switch, J3 AudioJack3_Ground_Switch, J4 AudioJack3_Ground_Switch, J5 Conn_02x03_Odd_Even, J6 Conn_02x03_Odd_Even, J7 Conn_02x05_Odd_Even, J8 Conn_01x03, J9 Conn_01x03

Commit message: Getting closer on jack board
Parts:
- moved J9 85.1 mm to (202.8, 75.8)
- moved J5 71.5 mm to (189.5, 78.3), turned to 90 degrees
- moved J6 37.1 mm to (162.2, 78.3), turned to 90 degrees
- moved J7 16.5 mm to (174.2, 78.3), turned to 90 degrees
- moved J4 14.3 mm to (200.8, 54.1)
- moved J3 13.8 mm to (180.3, 54.1)
- moved J2 13.4 mm to (159.8, 54.1)
- moved J1 13.0 mm to (139.2, 54.1)
- moved J8 7.64 mm to (147.8, 75.8)
Routing:
- net OUTL-R: track 0.00 -> 14.5 mm
- net OUTR-R: track 0.00 -> 13.7 mm
- net OUTL-T: track 0.00 -> 12.5 mm
- net OUTR-T: track 0.00 -> 11.8 mm
- net INL-T: track 0.00 -> 4.22 mm
- net INR-T: track 0.00 -> 3.16 mm
- net INL-R: track 0.00 -> 1.77 mm
- net INR-R: track 0.00 -> 1.22 mm
Other:
- board outline added: 93.2 x 49 mm
